File: kicad/chocV/chocV-top.kicad_pcb (KiCad board)
At the start: 2 copper layers, 36.8 x 47.9 mm, 6 parts

Commit message: new gerbers added
Parts:
- moved G*** 3.00 mm to (110.0, 68.6)
Changed lines of the file:
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@@
     (pad "1" thru_hole circle (at 0 -1.65) (size 0.7 0.7) (drill 0.4) (layers "*.Cu" "*.Mask")
       (net 2 "Net-(H2-Pad1)"))
-    (pad "1" thru_hole circle (at 0 0) (size 4.4 4.4) (drill 2.2) (layers "*.Cu" "*.Mask")
+    (pad "1" thru_hole circle (at 0 0.1) (size 4.4 4.4) (drill 2.2) (layers "*.Cu" "*.Mask")
       (net 2 "Net-(H2-Pad1)"))
     (pad "1" thru_hole circle (at 0 1.65) (size 0.7 0.7) (drill 0.4) (layers "*.Cu" "*.Mask")
@@
   )
   (footprint "KeebGraphics:HappyShigeoSilk" (layer "F.Cu")
-    (at 110 65.56)
+    (at 110 68.56)
     (attr board_only exclude_from_pos_files exclude_from_bom)
     (fp_text reference "G***" (at 0 0) (layer "F.SilkS") hide
